Commit message: Updated lab description package

File: src/lab_description/urdf/lab.urdf.xacro (robot description, xacro)
@@ -93,5 +93,5 @@
     trajectory_port="$(arg trajectory_port)"
     >
-    <origin xyz="0 0 0" rpy="0 0 0" />          <!-- robot position (relative to table in this case) -->
+    <origin xyz="0 0 0" rpy="0 0 -1.5708" />          <!-- robot position (relative to table in this case) -->
   </xacro:ur_robot>
   <xacro:if value="$(arg sim_gazebo)">
