Commit message: Updated table URDF with the new meshes

File: src/lab_description/urdf/table_macro.xacro (robot description, xacro)
@@ -4,21 +4,18 @@
     <link name="table">
       <inertial>
-        <origin xyz="-4.549932131044825e-16 -1.0237347294850857e-15 0.7364615189197282" rpy="0 0 0"/>
-        <mass value="321.36225333333357"/>
-        <inertia ixx="44.01548" iyy="24.813896" izz="57.996291" ixy="-0.0" iyz="-0.0" ixz="-0.0"/>
+        <origin xyz="0.29488015160583136 -0.0112575599024666 0.44349678570471823" rpy="0 0 0"/>
+        <mass value="67.19569705839687"/>
+        <inertia ixx="12.563401" iyy="9.982349" izz="11.832457" ixy="-0.068036" iyz="-0.075582" ixz="0.019671"/>
       </inertial>
       <visual>
-        <origin xyz="0.3385 0 0" rpy="0 0 0"/>
+        <origin xyz="0 0 0" rpy="0 0 0"/>
         <geometry>
-          <mesh filename="file://$(find lab_description)/meshes/table/table_demo.stl" scale="0.001 0.001 0.001"/>
+          <mesh filename="file://$(find lab_description)/meshes/ral_table/table.dae" scale="1.0 1.0 1.0"/>
         </geometry>
-        <material name="silver">
-          <color rgba="0.700 0.700 0.700 1.000"/>
-        </material>
       </visual>
       <collision>
-        <origin xyz="0.3385 0 0" rpy="0 0 0"/>
+        <origin xyz="0 0 0" rpy="0 0 0"/>
         <geometry>
-          <mesh filename="file://$(find lab_description)/meshes/table/table_demo.stl" scale="0.001 0.001 0.001"/>
+          <mesh filename="file://$(find lab_description)/meshes/ral_table/table_collision.dae" scale="1.0 1.0 1.0"/>
         </geometry>
       </collision>
@@ -32,5 +29,5 @@
       <parent link="table"/>
       <child link="table_child_mount"/>
-      <origin xyz="0 0 0.766" rpy="0 0 0"/>
+      <origin xyz="0 0 0.740" rpy="0 0 0"/>
     </joint>
   </xacro:macro>
